Commit message: add adapter and gripper to ur, work in gazebo

File: src/robot_setup/ur_robotiq_rs_description/urdf/test.urdf (robot description, URDF)
Before this commit: robot ur_robotiq_rs, 13 links, 12 joints
Links:
- added link gripper_mount_link
- added link ur_to_robotiq_link, mass 0.01; collision mesh filename=package://robotiq_description/meshes/collision/2f_85/ur_to_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; visual mesh filename=package://robotiq_description/meshes/visual/2f_85/ur_to_rob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
Joints:
- added joint gripper_side_joint: type fixed, parent ur_to_robotiq_link, child gripper_mount_link, origin xyz=0 0 0.011 rpy=0 0 0
- added joint ur_to_robotiq_joint: type fixed, parent tool0, child ur_to_robotiq_link, origin xyz=0 0 0 rpy=0 0 0.0
- joint base_joint: origin xyz=0 0 0 rpy=0 0 0 -> xyz=0 0.5 1.03 rpy=0 0 0

File: src/robot_setup/ur_robotiq_rs_description/urdf/ur_robotiq_rs.urdf.xacro (robot description, xacro)
@@ -1,10 +1,35 @@
 <?xml version="1.0"?>
 <robot xmlns:xacro="http://www.ros.org/wiki/xacro" name="ur_robotiq_rs">
+    <!-- parameters -->
+    <xacro:arg name="tf_prefix" default=""/>
+    <xacro:arg name="ur_type" default="ur5e"/>
+    <xacro:arg name="sim_gazebo" default="true" />
+    <xacro:arg name="simulation_controllers" default="$(find ur_robotiq_rs_description)/config/controllers.yaml" />
+    <xacro:arg name="initial_positions_file" default="$(find ur_robotiq_rs_description)/config/initial_positions.yaml"/>
+    <!-- import main macro -->
+    <xacro:include filename="$(find ur_robotiq_rs_description)/urdf/ur_robotiq_rs_macro.urdf.xacro"/>
     <link name="world"/>
-    <xacro:include filename="$(find ur_robotiq_rs_description)/urdf/ur_robotiq_rs_macro.urdf.xacro"/>
-    <xacro:ur_robotiq_rs name="ur" tf_prefix="" parent="world">
-        <xacro:arg name="ur_type" default="ur5e"/>
-        <xacro:arg name="initial_positions_file" default="$(find ur_robotiq_rs_description)/config/initial_positions.yaml"/>
+    <!-- robot: ur_robotiq_rs -->
+    <xacro:ur_robotiq_rs
+        ur_name="ur"
+        ur_type="$(arg ur_type)"
+        tf_prefix="$(arg tf_prefix)"
+        parent="world"
+        sim_gazebo="$(arg sim_gazebo)"
+        initial_positions="$(arg initial_positions_file)"
+        simulation_controllers="$(arg simulation_controllers)">
         <origin xyz="0 0.5 1.03" rpy="0 0 0" />
     </xacro:ur_robotiq_rs>
+    <xacro:if value="$(arg sim_gazebo)">
+        <gazebo reference="world">
+        </gazebo>
+        <xacro:if value="$(arg sim_gazebo)">
+            <!-- Gazebo plugins -->
+            <gazebo>
+                <plugin filename="libgazebo_ros2_control.so" name="gazebo_ros2_control">
+                    <parameters>$(arg simulation_controllers)</parameters>
+                </plugin>
+            </gazebo>
+          </xacro:if>
+    </xacro:if>
 </robot>

File: src/robot_setup/ur_robotiq_rs_description/urdf/ur_robotiq_rs_macro.urdf.xacro (robot description, xacro)
@@ -2,117 +2,111 @@
 <robot xmlns:xacro="http://wiki.ros.org/xacro">
   <xacro:macro name="ur_robotiq_rs" params="
-    name
+    ur_name:=ur
+    ur_type:=ur5x
     tf_prefix
     parent
-    *origin">
-    <!-- robot name parameter -->
-    <xacro:arg name="name" default="ur"/>
+    *origin
+    use_fake_hardware:=false
+    fake_sensor_commands:=false
+    sim_gazebo:=false
+    sim_ignition:=false
+    headless_mode:=false
+    initial_positions
+    simulation_controllers"
+    >
     <!-- import main macro -->
     <xacro:include filename="$(find ur_description)/urdf/ur_macro.xacro"/>
     <xacro:include filename="$(find robotiq_description)/urdf/robotiq_2f_85_macro.urdf.xacro" />
-    <!-- possible 'ur_type' values: ur3, ur3e, ur5, ur5e, ur10, ur10e, ur16e, ur20 -->
-    <!-- the default value should raise an error in case this was called without defining the type -->
-    <xacro:arg name="ur_type" default="ur5x"/>
-    <!-- parameters -->
-    <xacro:arg name="tf_prefix" default="" />
-    <xacro:arg name="joint_limit_params" default="$(find ur_description)/config/$(arg ur_type)/joint_limits.yaml"/>
-    <xacro:arg name="kinematics_params" default="$(find ur_description)/config/$(arg ur_type)/default_kinematics.yaml"/>
-    <xacro:arg name="physical_params" default="$(find ur_description)/config/$(arg ur_type)/physical_parameters.yaml"/>
-    <xacro:arg name="visual_params" default="$(find ur_description)/config/$(arg ur_type)/visual_parameters.yaml"/>
-    <xacro:arg name="transmission_hw_interface" default=""/>
-    <xacro:arg name="safety_limits" default="false"/>
-    <xacro:arg name="safety_pos_margin" default="0.15"/>
-    <xacro:arg name="safety_k_position" default="20"/>
+    <xacro:include filename="$(find robotiq_description)/urdf/ur_to_robotiq_adapter.urdf.xacro" />
+    <!-- property -->
+    <xacro:property name="joint_limits_parameters_file" value="$(find ur_description)/config/${ur_type}/joint_limits.yaml"/>
+    <xacro:property name="kinematics_parameters_file" value="$(find ur_description)/config/${ur_type}/default_kinematics.yaml"/>
+    <xacro:property name="physical_parameters_file" value="$(find ur_description)/config/${ur_type}/physical_parameters.yaml"/>
+    <xacro:property name="visual_parameters_file" value="$(find ur_description)/config/${ur_type}/visual_parameters.yaml"/>
+    <xacro:property name="transmission_hw_interface" value=""/>
+    <xacro:property name="safety_limits" value="false"/>
+    <xacro:property name="safety_pos_margin" value="0.15"/>
+    <xacro:property name="safety_k_position" value="20"/>
     <!-- ros2_control related parameters -->
-    <xacro:arg name="headless_mode" default="false" />
-    <xacro:arg name="robot_ip" default="0.0.0.0" />
-    <xacro:arg name="script_filename" default=""/>
-    <xacro:arg name="output_recipe_filename" default=""/>
-    <xacro:arg name="input_recipe_filename" default=""/>
-    <xacro:arg name="reverse_ip" default="0.0.0.0"/>
-    <xacro:arg name="script_command_port" default="50004"/>
-    <xacro:arg name="reverse_port" default="50001"/>
-    <xacro:arg name="script_sender_port" default="50002"/>
-    <xacro:arg name="trajectory_port" default="50003"/>
+    <xacro:property name="headless_mode" value="false" />
+    <xacro:property name="robot_ip" value="0.0.0.0" />
+    <xacro:property name="script_filename" value=""/>
+    <xacro:property name="output_recipe_filename" value=""/>
+    <xacro:property name="input_recipe_filename" value=""/>
+    <xacro:property name="reverse_ip" value="0.0.0.0"/>
+    <xacro:property name="script_command_port" value="50004"/>
+    <xacro:property name="reverse_port" value="50001"/>
+    <xacro:property name="script_sender_port" value="50002"/>
+    <xacro:property name="trajectory_port" value="50003"/>
     <!--   tool communication related parameters-->
-    <xacro:arg name="use_tool_communication" default="false" />
-    <xacro:arg name="tool_voltage" default="0" />
-    <xacro:arg name="tool_parity" default="0" />
-    <xacro:arg name="tool_baud_rate" default="115200" />
-    <xacro:arg name="tool_stop_bits" default="1" />
-    <xacro:arg name="tool_rx_idle_chars" default="1.5" />
-    <xacro:arg name="tool_tx_idle_chars" default="3.5" />
-    <xacro:arg name="tool_device_name" default="/tmp/ttyUR" />
-    <xacro:arg name="tool_tcp_port" default="54321" />
-      <!-- Simulation parameters -->
+    <xacro:property name="use_tool_communication" value="false" />
+    <xacro:property name="tool_voltage" value="0" />
+    <xacro:property name="tool_parity" value="0" />
+    <xacro:property name="tool_baud_rate" value="115200" />
+    <xacro:property name="tool_stop_bits" value="1" />
+    <xacro:property name="tool_rx_idle_chars" value="1.5" />
+    <xacro:property name="tool_tx_idle_chars" value="3.5" />
+    <xacro:property name="tool_device_name" value="/tmp/ttyUR" />
+    <xacro:property name="tool_tcp_port" value="54321" />
+    <!-- Simulation parameters -->
     <xacro:arg name="use_fake_hardware" default="false" />
     <xacro:arg name="fake_sensor_commands" default="false" />
-    <xacro:arg name="sim_gazebo" default="true" />
+    <xacro:arg name="sim_gazebo" default="false" />
     <xacro:arg name="sim_ignition" default="false" />
     <xacro:arg name="simulation_controllers" default="" />
-    <!-- initial position for simulations (Fake Hardware, Gazebo, Ignition) -->
-    <xacro:arg name="initial_positions_file" default="$(find ur_description)/config/initial_positions.yaml"/>
-    <xacro:arg name="parent_link" default="world"/>
-    <!-- convert to property to use substitution in function -->
-    <xacro:property name="initial_positions_file" default="$(arg initial_positions_file)"/>
     <!-- arm -->
     <xacro:ur_robot
-      name="$(arg name)"
-      tf_prefix="$(arg tf_prefix)"
-      parent="$(arg parent_link)"
-      joint_limits_parameters_file="$(arg joint_limit_params)"
-      kinematics_parameters_file="$(arg kinematics_params)"
-      physical_parameters_file="$(arg physical_params)"
-      visual_parameters_file="$(arg visual_params)"
-      transmission_hw_interface="$(arg transmission_hw_interface)"
-      safety_limits="$(arg safety_limits)"
-      safety_pos_margin="$(arg safety_pos_margin)"
-      safety_k_position="$(arg safety_k_position)"
-      use_fake_hardware="$(arg use_fake_hardware)"
-      fake_sensor_commands="$(arg fake_sensor_commands)"
-      sim_gazebo="$(arg sim_gazebo)"
-      sim_ignition="$(arg sim_ignition)"
-      headless_mode="$(arg headless_mode)"
-      initial_positions="${xacro.load_yaml(initial_positions_file)}"
-      use_tool_communication="$(arg use_tool_communication)"
-      tool_voltage="$(arg tool_voltage)"
-      tool_parity="$(arg tool_parity)"
-      tool_baud_rate="$(arg tool_baud_rate)"
-      tool_stop_bits="$(arg tool_stop_bits)"
-      tool_rx_idle_chars="$(arg tool_rx_idle_chars)"
-      tool_tx_idle_chars="$(arg tool_tx_idle_chars)"
-      tool_device_name="$(arg tool_device_name)"
-      tool_tcp_port="$(arg tool_tcp_port)"
-      robot_ip="$(arg robot_ip)"
-      script_filename="$(arg script_filename)"
-      output_recipe_filename="$(arg output_recipe_filename)"
-      input_recipe_filename="$(arg input_recipe_filename)"
-      reverse_ip="$(arg reverse_ip)"
-      script_command_port="$(arg script_command_port)"
-      reverse_port="$(arg reverse_port)"
-      script_sender_port="$(arg script_sender_port)"
-      trajectory_port="$(arg trajectory_port)"
+      name="${ur_name}"
+      tf_prefix="${tf_prefix}"
+      parent="${parent}"
+      joint_limits_parameters_file="${joint_limits_parameters_file}"
+      kinematics_parameters_file="${kinematics_parameters_file}"
+      physical_parameters_file="${physical_parameters_file}"
+      visual_parameters_file="${visual_parameters_file}"
+      transmission_hw_interface="${transmission_hw_interface}"
+      safety_limits="${safety_limits}"
+      safety_pos_margin="${safety_pos_margin}"
+      safety_k_position="${safety_k_position}"
+      use_fake_hardware="${use_fake_hardware}"
+      fake_sensor_commands="${fake_sensor_commands}"
+      sim_gazebo="${sim_gazebo}"
+      sim_ignition="${sim_ignition}"
+      headless_mode="${headless_mode}"
+      initial_positions="${xacro.load_yaml(initial_positions)}"
+      use_tool_communication="${use_tool_communication}"
+      tool_voltage="${tool_voltage}"
+      tool_parity="${tool_parity}"
+      tool_baud_rate="${tool_baud_rate}"
+      tool_stop_bits="${tool_stop_bits}"
+      tool_rx_idle_chars="${tool_rx_idle_chars}"
+      tool_tx_idle_chars="${tool_tx_idle_chars}"
+      tool_device_name="${tool_device_name}"
+      tool_tcp_port="${tool_tcp_port}"
+      robot_ip="${robot_ip}"
+      script_filename="${script_filename}"
+      output_recipe_filename="${output_recipe_filename}"
+      input_recipe_filename="${input_recipe_filename}"
+      reverse_port="${reverse_port}"
+      script_sender_port="${script_sender_port}"
+      reverse_ip="${reverse_ip}"
+      script_command_port="${script_command_port}"
+      trajectory_port="${trajectory_port}"
       >
-      <origin xyz="0 0 0" rpy="0 0 0" />          <!-- position robot in the parent link -->
+      <xacro:insert_block name="origin" />          <!-- position robot in the parent link -->
     </xacro:ur_robot>
-    <xacro:if value="$(arg sim_gazebo)">
-      <!-- Gazebo plugins -->
-      <gazebo>
-        <plugin filename="libgazebo_ros2_control.so" name="$(arg tf_prefix)ur_gazebo_ros2_control">
-          <parameters>$(arg simulation_controllers)</parameters>
-        </plugin>
-      </gazebo>
-    </xacro:if>
-    <xacro:if value="$(arg sim_ignition)">
-      <!-- Gazebo plugins -->
-      <gazebo reference="world">
-      </gazebo>
-      <gazebo>
-        <plugin filename="libign_ros2_control-system.so" name="ign_ros2_control::IgnitionROS2ControlPlugin">
-          <parameters>$(arg simulation_controllers)</parameters>
-          <controller_manager_node_name>$(arg tf_prefix)controller_manager</controller_manager_node_name>
-        </plugin>
-      </gazebo>
-    </xacro:if>
+    <!-- adapter -->
+    <xacro:ur_to_robotiq
+      prefix="${tf_prefix}"
+      connected_to="${tf_prefix}tool0"
+      rotation="0.0"
+      />
+    <!-- gripper -->
+    <xacro:robotiq_2f_85_gripper name="RobotiqGripperHardwareInterface"
+        prefix="${tf_prefix}"
+        parent="${tf_prefix}gripper_mount_link"
+        use_fake_hardware="$(arg use_fake_hardware)"
+        sim_gazebo="$(arg sim_gazebo)">
+        <origin xyz="0 0 0" rpy="0 0 0" />
+    </xacro:robotiq_2f_85_gripper>
   </xacro:macro>
 </robot>
