Commit message: add realsense to the robot

File: src/robot_setup/ur_robotiq_rs_description/srdf/ur_robotiq_rs_macro.srdf.xacro (robot description, xacro)
@@ -9,4 +9,8 @@
         <!-- robotiq 2f 85 -->
         <xacro:robotiq_2f_85_srdf prefix="${prefix}"/>
+        <group name="ur_robotiq">
+            <group name="ur_manipulator"/>
+            <group name="robotiq_2f_85_gripper"/>
+        </group>
         <!--DISABLE COLLISIONS By default it is assumed that any link of the robot could potentially come into collision with any other link in the robot. This tag disables collision checking between a specified pair of links. -->
         <disable_collisions link1="${prefix}robotiq_85_base_link" link2="${prefix}ur_to_robotiq_link" reason="Adjacent"/>

File: src/robot_setup/ur_robotiq_rs_description/urdf/test.urdf (robot description, URDF)
Before this commit: robot ur_robotiq_rs, 15 links, 14 joints
Links:
- added link dummy_child1
- added link dummy_child2
- added link dummy_child3
- added link dummy_child4
- added link dummy_child5
- added link robotiq_85_base_link, mass 6.6320197e-01; collision mesh filename=file:///home/xiaobaige/ur_project_ros2/install/robotiq_desc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; visual mesh filename=file:///home/xiaobaige/ur_project_ros2/install/robotiq_desc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
- added link robotiq_85_left_finger_link, mass 4.260376752e-02; collision mesh filename=file:///home/xiaobaige/ur_project_ros2/install/robotiq_desc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; visual mesh filename=file:///home/xiaobaige/ur_project_ros2/install/robotiq_desc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
- added link robotiq_85_left_finger_tip_link, mass 4.268588744e-02; collision mesh filename=file:///home/xiaobaige/ur_project_ros2/install/robotiq_desc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; visual mesh filename=file:///home/xiaobaige/ur_project_ros2/install/robotiq_desc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
- added link robotiq_85_left_inner_knuckle_link, mass 2.969376448e-02; collision mesh filename=file:///home/xiaobaige/ur_project_ros2/install/robotiq_desc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; visual mesh filename=file:///home/xiaobaige/ur_project_ros2/install/robotiq_desc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
- added link robotiq_85_left_knuckle_link, mass 1.384773208e-02; collision mesh filename=file:///home/xiaobaige/ur_project_ros2/install/robotiq_desc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; visual mesh filename=file:///home/xiaobaige/ur_project_ros2/install/robotiq_desc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
- added link robotiq_85_right_finger_link, mass 4.260376752000000e-02; collision mesh filename=file:///home/xiaobaige/ur_project_ros2/install/robotiq_desc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; visual mesh filename=file:///home/xiaobaige/ur_project_ros2/install/robotiq_desc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
- added link robotiq_85_right_finger_tip_link, mass 4.268588744e-02; collision mesh filename=file:///home/xiaobaige/ur_project_ros2/install/robotiq_desc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; visual mesh filename=file:///home/xiaobaige/ur_project_ros2/install/robotiq_desc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
- added link robotiq_85_right_inner_knuckle_link, mass 2.969376448e-02; collision mesh filename=file:///home/xiaobaige/ur_project_ros2/install/robotiq_desc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; visual mesh filename=file:///home/xiaobaige/ur_project_ros2/install/robotiq_desc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
- added link robotiq_85_right_knuckle_link, mass 1.384773208e-02; collision mesh filename=file:///home/xiaobaige/ur_project_ros2/install/robotiq_desc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; visual mesh filename=file:///home/xiaobaige/ur_project_ros2/install/robotiq_desc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
- link ur_to_robotiq_link: geometry collision mesh filename=file:///home/xiaobaige/ur_project_ros2/install/robotiq_desc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; visual mesh filename=file:///home/xiaobaige/ur_project_ros2/install/robotiq_desc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
Joints:
- added joint robotiq_85_base_joint: type fixed, parent gripper_mount_link, child robotiq_85_base_link, origin xyz=0 0 0 rpy=0 0 0
- added joint robotiq_85_left_finger_joint: type fixed, parent robotiq_85_left_knuckle_link, child robotiq_85_left_finger_link, origin xyz=0.03152616 0.0 -0.00376347 rpy=0 0 0
- added joint robotiq_85_left_finger_tip_joint: type continuous, parent robotiq_85_left_finger_link, child robotiq_85_left_finger_tip_link, origin xyz=0.00563134 0.0 0.04718515 rpy=0 0 0, axis 0 -1 0, mimic joint=robotiq_85_left_knuckle_joint multiplier=-1
- added joint robotiq_85_left_finger_tip_joint_mimic: type fixed, parent robotiq_85_base_link, child dummy_child4
- added joint robotiq_85_left_inner_knuckle_joint: type continuous, parent robotiq_85_base_link, child robotiq_85_left_inner_knuckle_link, origin xyz=0.0127 0.0 0.06142 rpy=0 0 0, axis 0 -1 0, mimic joint=robotiq_85_left_knuckle_joint
- added joint robotiq_85_left_inner_knuckle_joint_mimic: type fixed, parent robotiq_85_base_link, child dummy_child2
- added joint robotiq_85_left_knuckle_joint: type revolute, parent robotiq_85_base_link, child robotiq_85_left_knuckle_link, origin xyz=0.03060114 0.0 0.05490452 rpy=0 0 0, axis 0 -1 0, limit lower=0.0 upper=0.8 effort=50 velocity=0.5
- added joint robotiq_85_right_finger_joint: type fixed, parent robotiq_85_right_knuckle_link, child robotiq_85_right_finger_link, origin xyz=-0.03152616 0.0 -0.00376347 rpy=0 0 0
- added joint robotiq_85_right_finger_tip_joint: type continuous, parent robotiq_85_right_finger_link, child robotiq_85_right_finger_tip_link, origin xyz=-0.00563134 0.0 0.04718515 rpy=0 0 0, axis 0 -1 0, mimic joint=robotiq_85_left_knuckle_joint
- added joint robotiq_85_right_finger_tip_joint_mimic: type fixed, parent robotiq_85_base_link, child dummy_child5
- added joint robotiq_85_right_inner_knuckle_joint: type continuous, parent robotiq_85_base_link, child robotiq_85_right_inner_knuckle_link, origin xyz=-0.0127 0.0 0.06142 rpy=0 0 0, axis 0 -1 0, mimic joint=robotiq_85_left_knuckle_joint multiplier=-1
- added joint robotiq_85_right_inner_knuckle_joint_mimic: type fixed, parent robotiq_85_base_link, child dummy_child3
- added joint robotiq_85_right_knuckle_joint: type revolute, parent robotiq_85_base_link, child robotiq_85_right_knuckle_link, origin xyz=-0.03060114 0.0 0.05490452 rpy=0 0 0, axis 0 -1 0, limit lower=-0.8 upper=0.0 effort=50 velocity=0.5, mimic joint=robotiq_85_left_knuckle_joint multiplier=-1
- added joint robotiq_85_right_knuckle_joint_mimic: type fixed, parent robotiq_85_base_link, child dummy_child1

File: src/robot_setup/ur_robotiq_rs_description/urdf/ur_robotiq_rs.urdf.xacro (robot description, xacro)
@@ -4,5 +4,5 @@
     <xacro:arg name="tf_prefix" default=""/>
     <xacro:arg name="ur_type" default="ur5e"/>
-    <xacro:arg name="sim_gazebo" default="false" />
+    <xacro:arg name="sim_gazebo" default="true" />
     <xacro:arg name="simulation_controllers" default="$(find ur_robotiq_rs_description)/config/controllers.yaml" />
     <xacro:arg name="initial_positions_file" default="$(find ur_robotiq_rs_description)/config/initial_positions.yaml"/>

File: src/robot_setup/ur_robotiq_rs_description/urdf/ur_robotiq_rs_macro.urdf.xacro (robot description, xacro)
@@ -19,4 +19,5 @@
     <xacro:include filename="$(find robotiq_description)/urdf/robotiq_2f_85_macro.urdf.xacro" />
     <xacro:include filename="$(find robotiq_description)/urdf/ur_to_robotiq_adapter.urdf.xacro" />
+    <xacro:include filename="$(find ur_robotiq_rs_description)/urdf/realsense_d435.urdf.xacro"/>
     <!-- property -->
     <xacro:property name="joint_limits_parameters_file" value="$(find ur_description)/config/${ur_type}/joint_limits.yaml"/>
@@ -109,4 +110,13 @@
         <origin xyz="0 0 0" rpy="0 0 0" />
     </xacro:robotiq_2f_85_gripper>
+    <!-- realsense camera -->
+    <!-- Use the nominal extrinsics between camera frames if the calibrated extrinsics aren't being published. e.g. running the device in simulation  -->
+    <xacro:sensor_d435 parent="${tf_prefix}tool0"
+      name="${tf_prefix}camera"
+      use_nominal_extrinsics="true"
+      add_plug="false"
+      use_mesh="true">
+      <origin xyz="0 -0.1 0" rpy="0 -1.5707 1.5707"/>
+    </xacro:sensor_d435>
   </xacro:macro>
 </robot>

Commit message: add ur_robotiq_rs helper node

File: src/robot_setup/ur_robotiq_rs_description/srdf/ur_robotiq_rs_macro.srdf.xacro (robot description, xacro)
@@ -13,4 +13,12 @@
             <group name="robotiq_2f_85_gripper"/>
         </group>
+        <group_state name="${prefix}ready" group="${prefix}ur_manipulator">
+            <joint name="${prefix}elbow_joint" value="1.5707" />
+            <joint name="${prefix}shoulder_lift_joint" value="-1.5707" />
+            <joint name="${prefix}shoulder_pan_joint" value="0" />
+            <joint name="${prefix}wrist_1_joint" value="-1.5707" />
+            <joint name="${prefix}wrist_2_joint" value="-1.5707" />
+            <joint name="${prefix}wrist_3_joint" value="0" />
+        </group_state>
         <!--DISABLE COLLISIONS By default it is assumed that any link of the robot could potentially come into collision with any other link in the robot. This tag disables collision checking between a specified pair of links. -->
         <disable_collisions link1="${prefix}robotiq_85_base_link" link2="${prefix}ur_to_robotiq_link" reason="Adjacent"/>

File: src/robot_setup/ur_robotiq_rs_description/urdf/ur_robotiq_rs.urdf.xacro (robot description, xacro)
@@ -7,4 +7,7 @@
     <xacro:arg name="simulation_controllers" default="$(find ur_robotiq_rs_description)/config/controllers.yaml" />
     <xacro:arg name="initial_positions_file" default="$(find ur_robotiq_rs_description)/config/initial_positions.yaml"/>
+    <xacro:arg name="base_frame_file" default="$(find ur_robotiq_rs_description)/config/base_frame.yaml" />
+    <xacro:property name="base_frame_file" value="$(arg base_frame_file)"/>
+    <xacro:property name="base_frame" value="${xacro.load_yaml(base_frame_file)['base_frame']}"/>
     <!-- import main macro -->
     <xacro:include filename="$(find ur_robotiq_rs_description)/urdf/ur_robotiq_rs_macro.urdf.xacro"/>
@@ -19,5 +22,6 @@
         initial_positions="$(arg initial_positions_file)"
         simulation_controllers="$(arg simulation_controllers)">
-        <origin xyz="0 0.5 1.03" rpy="0 0 0" />
+        <origin xyz="${base_frame['x']} ${base_frame['y']} ${base_frame['z']}"
+            rpy="${base_frame['roll']} ${base_frame['pitch']} ${base_frame['yaw']}" />
     </xacro:ur_robotiq_rs>
     <xacro:if value="$(arg sim_gazebo)">
