Commit message: adjust grasp fix loading

File: src/robot_setup/dual_ur_robotiq_rs_description/urdf/dual_ur_robotiq_rs.urdf.xacro (robot description, xacro)
@@ -37,12 +37,42 @@
         <gazebo reference="world">
         </gazebo>
-        <xacro:if value="$(arg sim_gazebo)">
-            <!-- Gazebo plugins -->
-            <gazebo>
-                <plugin filename="libgazebo_ros2_control.so" name="gazebo_ros2_control">
-                    <parameters>$(arg simulation_controllers)</parameters>
-                </plugin>
-            </gazebo>
-          </xacro:if>
+        <!-- Gazebo plugins -->
+        <gazebo>
+            <plugin filename="libgazebo_ros2_control.so" name="gazebo_ros2_control">
+                <parameters>$(arg simulation_controllers)</parameters>
+            </plugin>
+        </gazebo>
+        <gazebo>
+            <!-- grasp fix plugin for gazebo classic -->
+            <plugin name="gazebo_grasp_fix" filename="libgazebo_grasp_fix.so">
+                <arm>
+                    <arm_name>left_robotiq_85_gripper_arm</arm_name>
+                    <palm_link>left_wrist_3_link</palm_link>
+                    <gripper_link>left_robotiq_85_left_finger_tip_link</gripper_link>
+                    <gripper_link>left_robotiq_85_right_finger_tip_link</gripper_link>
+                    <gripper_link>left_robotiq_85_left_knuckle_link</gripper_link>
+                    <gripper_link>left_robotiq_85_right_knuckle_link</gripper_link>
+                    <gripper_link>left_robotiq_85_left_inner_knuckle_link</gripper_link>
+                    <gripper_link>left_robotiq_85_right_inner_knuckle_link</gripper_link>
+                </arm>
+                <arm>
+                    <arm_name>right_robotiq_85_gripper_arm</arm_name>
+                    <palm_link>right_wrist_3_link</palm_link>
+                    <gripper_link>right_robotiq_85_left_finger_tip_link</gripper_link>
+                    <gripper_link>right_robotiq_85_right_finger_tip_link</gripper_link>
+                    <gripper_link>right_robotiq_85_left_knuckle_link</gripper_link>
+                    <gripper_link>right_robotiq_85_right_knuckle_link</gripper_link>
+                    <gripper_link>right_robotiq_85_left_inner_knuckle_link</gripper_link>
+                    <gripper_link>right_robotiq_85_right_inner_knuckle_link</gripper_link>
+                </arm>
+                <forces_angle_tolerance>150</forces_angle_tolerance>
+                <update_rate>30</update_rate>
+                <grip_count_threshold>1</grip_count_threshold>
+                <max_grip_count>2</max_grip_count>
+                <release_tolerance>0.01</release_tolerance>
+                <disable_collisions_on_attach>false</disable_collisions_on_attach>
+                <contact_topic>__default_topic__</contact_topic>
+             </plugin>
+         </gazebo>
     </xacro:if>
 </robot>

File: src/robot_setup/dual_ur_robotiq_rs_description/urdf/test.urdf (robot description, URDF)
Before this commit: robot dual_ur_robotiq_rs, 77 links, 76 joints
Links:
- link left_camera_link: geometry collision box size=0.02505 0.09 0.025; visual mesh filename=file:///opt/ros/humble/share/realsense2_description/meshes/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
- link right_camera_link: geometry collision box size=0.02505 0.09 0.025; visual mesh filename=file:///opt/ros/humble/share/realsense2_description/meshes/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

File: src/robot_setup/ur_robotiq_rs_description/urdf/realsense_d435.gazebo.xacro (robot description, xacro)
@@ -117,12 +117,12 @@
       	<colorUpdateRate>30.0</colorUpdateRate>
       	<infraredUpdateRate>1.0</infraredUpdateRate>
-      	<depthTopicName>depth/image_raw</depthTopicName>
-      	<depthCameraInfoTopicName>depth/camera_info</depthCameraInfoTopicName>
-      	<colorTopicName>color/image_raw</colorTopicName>
-      	<colorCameraInfoTopicName>color/camera_info</colorCameraInfoTopicName>
-      	<infrared1TopicName>infra1/image_raw</infrared1TopicName>
-      	<infrared1CameraInfoTopicName>infra1/camera_info</infrared1CameraInfoTopicName>
-      	<infrared2TopicName>infra2/image_raw</infrared2TopicName>
-      	<infrared2CameraInfoTopicName>infra2/camera_info</infrared2CameraInfoTopicName>
+      	<depthTopicName>${topics_ns}/${camera_name}/depth/image_raw</depthTopicName>
+      	<depthCameraInfoTopicName>${topics_ns}/${camera_name}/depth/camera_info</depthCameraInfoTopicName>
+      	<colorTopicName>${topics_ns}/${camera_name}/color/image_raw</colorTopicName>
+      	<colorCameraInfoTopicName>${topics_ns}/${camera_name}/color/camera_info</colorCameraInfoTopicName>
+      	<infrared1TopicName>${topics_ns}/${camera_name}/infra1/image_raw</infrared1TopicName>
+      	<infrared1CameraInfoTopicName>${topics_ns}/${camera_name}/infra1/camera_info</infrared1CameraInfoTopicName>
+      	<infrared2TopicName>${topics_ns}/${camera_name}/infra2/image_raw</infrared2TopicName>
+      	<infrared2CameraInfoTopicName>${topics_ns}/${camera_name}/infra2/camera_info</infrared2CameraInfoTopicName>
       	<colorOpticalframeName>${color_optical_frame}</colorOpticalframeName>
       	<depthOpticalframeName>${depth_optical_frame}</depthOpticalframeName>
@@ -132,5 +132,5 @@
       	<rangeMaxDepth>10.0</rangeMaxDepth>
       	<pointCloud>true</pointCloud>
-      	<pointCloudTopicName>depth/points</pointCloudTopicName>
+      	<pointCloudTopicName>${topics_ns}/${camera_name}/depth/points</pointCloudTopicName>
       	<pointCloudCutoff>0.5</pointCloudCutoff>
       </plugin>

File: src/robot_setup/ur_robotiq_rs_description/urdf/realsense_d435.urdf.xacro (robot description, xacro)
@@ -146,7 +146,7 @@
       <link name="${name}_color_optical_frame"/>
     </xacro:if>
-    <xacro:gazebo_d435 camera_name="${name}"
+    <xacro:gazebo_d435 camera_name="d435"
       reference_link="${name}_link"
-      topics_ns="{name}_d435"
+      topics_ns="${name}"
       depth_optical_frame="${name}_depth_optical_frame"
       color_optical_frame="${name}_color_optical_frame"

File: src/robot_setup/ur_robotiq_rs_description/urdf/test.urdf (robot description, URDF)
Before this commit: robot ur_robotiq_rs, 29 links, 28 joints
Links:
- added link camera_bottom_screw_frame
- added link camera_color_frame
- added link camera_color_optical_frame
- added link camera_depth_frame
- added link camera_depth_optical_frame
- added link camera_infra1_frame
- added link camera_infra1_optical_frame
- added link camera_infra2_frame
- added link camera_infra2_optical_frame
- added link camera_link, mass 0.072; collision box size=0.02505 0.09 0.025; visual mesh filename=file:///opt/ros/humble/share/realsense2_description/meshes/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
Joints:
- added joint camera_color_joint: type fixed, parent camera_link, child camera_color_frame, origin xyz=0 0.015 0 rpy=0 0 0
- added joint camera_color_optical_joint: type fixed, parent camera_color_frame, child camera_color_optical_frame, origin xyz=0 0 0 rpy=-1.5707963267948966 0 -1.5707963267948966
- added joint camera_depth_joint: type fixed, parent camera_link, child camera_depth_frame, origin xyz=0 0 0 rpy=0 0 0
- added joint camera_depth_optical_joint: type fixed, parent camera_depth_frame, child camera_depth_optical_frame, origin xyz=0 0 0 rpy=-1.5707963267948966 0 -1.5707963267948966
- added joint camera_infra1_joint: type fixed, parent camera_link, child camera_infra1_frame, origin xyz=0 0.0 0 rpy=0 0 0
- added joint camera_infra1_optical_joint: type fixed, parent camera_infra1_frame, child camera_infra1_optical_frame, origin xyz=0 0 0 rpy=-1.5707963267948966 0 -1.5707963267948966
- added joint camera_infra2_joint: type fixed, parent camera_link, child camera_infra2_frame, origin xyz=0 -0.05 0 rpy=0 0 0
- added joint camera_infra2_optical_joint: type fixed, parent camera_infra2_frame, child camera_infra2_optical_frame, origin xyz=0 0 0 rpy=-1.5707963267948966 0 -1.5707963267948966
- added joint camera_joint: type fixed, parent tool0, child camera_bottom_screw_frame, origin xyz=0 -0.1 0 rpy=0 -1.5707 1.5707
- added joint camera_link_joint: type fixed, parent camera_bottom_screw_frame, child camera_link, origin xyz=0.010600000000000002 0.0175 0.0125 rpy=0 0 0

File: src/robot_setup/ur_robotiq_rs_description/urdf/ur_robotiq_rs.urdf.xacro (robot description, xacro)
@@ -24,12 +24,32 @@
         <gazebo reference="world">
         </gazebo>
-        <xacro:if value="$(arg sim_gazebo)">
-            <!-- Gazebo plugins -->
-            <gazebo>
-                <plugin filename="libgazebo_ros2_control.so" name="gazebo_ros2_control">
-                    <parameters>$(arg simulation_controllers)</parameters>
-                </plugin>
-            </gazebo>
-          </xacro:if>
+        <!-- Gazebo plugins -->
+        <gazebo>
+            <plugin filename="libgazebo_ros2_control.so" name="gazebo_ros2_control">
+                <parameters>$(arg simulation_controllers)</parameters>
+            </plugin>
+        </gazebo>
+        <gazebo>
+            <!-- grasp fix plugin for gazebo classic -->
+            <plugin name="gazebo_grasp_fix" filename="libgazebo_grasp_fix.so">
+                <arm>
+                    <arm_name>$(arg tf_prefix)robotiq_85_gripper_arm</arm_name>
+                    <palm_link>$(arg tf_prefix)wrist_3_link</palm_link>
+                    <gripper_link>$(arg tf_prefix)robotiq_85_left_finger_tip_link</gripper_link>
+                    <gripper_link>$(arg tf_prefix)robotiq_85_right_finger_tip_link</gripper_link>
+                    <gripper_link>$(arg tf_prefix)robotiq_85_left_knuckle_link</gripper_link>
+                    <gripper_link>$(arg tf_prefix)robotiq_85_right_knuckle_link</gripper_link>
+                    <gripper_link>$(arg tf_prefix)robotiq_85_left_inner_knuckle_link</gripper_link>
+                    <gripper_link>$(arg tf_prefix)robotiq_85_right_inner_knuckle_link</gripper_link>
+                </arm>
+                <forces_angle_tolerance>150</forces_angle_tolerance>
+                <update_rate>30</update_rate>
+                <grip_count_threshold>1</grip_count_threshold>
+                <max_grip_count>2</max_grip_count>
+                <release_tolerance>0.01</release_tolerance>
+                <disable_collisions_on_attach>false</disable_collisions_on_attach>
+                <contact_topic>__default_topic__</contact_topic>
+             </plugin>
+         </gazebo>
     </xacro:if>
 </robot>

File: src/robot_setup/ur_robotiq_rs_description/urdf/ur_robotiq_rs_macro.urdf.xacro (robot description, xacro)
@@ -101,6 +101,5 @@
         parent="${tf_prefix}gripper_mount_link"
         use_fake_hardware="${use_fake_hardware}"
-        sim_gazebo="$(arg sim_gazebo)"
-        palm_link="${tf_prefix}wrist_3_link">
+        sim_gazebo="$(arg sim_gazebo)">
         <origin xyz="0 0 0" rpy="0 0 0" />
     </xacro:robotiq_2f_85_gripper>

Commit message: update dual_ur_robotiq_rs and add new task dual_plan

File: src/robot_setup/dual_ur_robotiq_rs_description/urdf/dual_ur_robotiq_rs.urdf.xacro (robot description, xacro)
@@ -7,4 +7,8 @@
     <xacro:arg name="left_initial_positions_file" default="$(find dual_ur_robotiq_rs_description)/config/left_initial_positions.yaml"/>
     <xacro:arg name="right_initial_positions_file" default="$(find dual_ur_robotiq_rs_description)/config/right_initial_positions.yaml"/>
+    <xacro:arg name="base_frame_file" default="$(find dual_ur_robotiq_rs_description)/config/base_frame.yaml" />
+    <xacro:property name="base_frame_file" value="$(arg base_frame_file)"/>
+    <xacro:property name="left_base_frame" value="${xacro.load_yaml(base_frame_file)['left_base_frame']}"/>
+    <xacro:property name="right_base_frame" value="${xacro.load_yaml(base_frame_file)['right_base_frame']}"/>
     <!-- import main macro -->
     <xacro:include filename="$(find ur_robotiq_rs_description)/urdf/ur_robotiq_rs_macro.urdf.xacro"/>
@@ -19,5 +23,6 @@
         initial_positions="$(arg left_initial_positions_file)"
         simulation_controllers="$(arg simulation_controllers)">
-        <origin xyz="0 0.5 1.03" rpy="0 0 0" />
+        <origin xyz="${left_base_frame['x']} ${left_base_frame['y']} ${left_base_frame['z']}"
+            rpy="${left_base_frame['roll']} ${left_base_frame['pitch']} ${left_base_frame['yaw']}" />
     </xacro:ur_robotiq_rs>
     <!-- This avoids the redefinition of materials in case multple cameras are imported. -->
@@ -32,5 +37,6 @@
         initial_positions="$(arg right_initial_positions_file)"
         simulation_controllers="$(arg simulation_controllers)">
-        <origin xyz="0 -0.5 1.03" rpy="0 0 0" />
+        <origin xyz="${right_base_frame['x']} ${right_base_frame['y']} ${right_base_frame['z']}"
+            rpy="${right_base_frame['roll']} ${right_base_frame['pitch']} ${right_base_frame['yaw']}" />
     </xacro:ur_robotiq_rs>
     <xacro:if value="$(arg sim_gazebo)">

File: src/robot_setup/dual_ur_robotiq_rs_description/urdf/test.urdf (robot description, URDF)
Before this commit: robot dual_ur_robotiq_rs, 77 links, 76 joints
Links:
- link left_camera_link: geometry collision box size=0.02505 0.09 0.025; visual mesh filename=file:///home/xiaobaige/ros2_ws/install/realsense2_descripti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
- link right_camera_link: geometry collision box size=0.02505 0.09 0.025; visual mesh filename=file:///home/xiaobaige/ros2_ws/install/realsense2_descripti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
Joints:
- joint left_base_joint: origin xyz=0 0.5 1.03 rpy=0 0 0 -> xyz=0.0 0.5 1.0 rpy=0.0 0.0 0.0
- joint right_base_joint: origin xyz=0 -0.5 1.03 rpy=0 0 0 -> xyz=0.0 -0.5 1.0 rpy=0.0 0.0 0.0

File: src/robot_setup/ur_robotiq_rs_description/srdf/ur_robotiq_rs_macro.srdf.xacro (robot description, xacro)
@@ -9,7 +9,7 @@
         <!-- robotiq 2f 85 -->
         <xacro:robotiq_2f_85_srdf prefix="${prefix}"/>
-        <group name="ur_robotiq">
-            <group name="ur_manipulator"/>
-            <group name="robotiq_2f_85_gripper"/>
+        <group name="${prefix}ur_robotiq">
+            <group name="${prefix}ur_manipulator"/>
+            <group name="${prefix}robotiq_2f_85_gripper"/>
         </group>
         <group_state name="${prefix}ready" group="${prefix}ur_manipulator">

File: src/robot_setup/ur_robotiq_rs_description/urdf/ur_robotiq_rs_macro.urdf.xacro (robot description, xacro)
@@ -104,4 +104,11 @@
         <origin xyz="0 0 0" rpy="0 0 0" />
     </xacro:robotiq_2f_85_gripper>
+    <!-- grasp point for planning -->
+    <link name="${tf_prefix}grasp_point"/>
+    <joint name="${tf_prefix}grasp_point_joint" type="fixed">
+      <parent link="${tf_prefix}tool0"/>
+      <child link="${tf_prefix}grasp_point"/>
+      <origin xyz="0 0 0.15" rpy="0 0 0"/>
+    </joint>
     <!-- realsense camera -->
     <!-- Use the nominal extrinsics between camera frames if the calibrated extrinsics aren't being published. e.g. running the device in simulation  -->
