Commit message: fix bug of xacro parsing

File: src/robot_setup/dual_ur_robotiq_rs_description/urdf/test.urdf (robot description, URDF)
Before this commit: robot dual_ur_robotiq_rs, 77 links, 76 joints
Links:
- added link left_grasp_point
- added link right_grasp_point
- link left_camera_link: geometry collision box size=0.02505 0.09 0.025; visual mesh filename=file:///opt/ros/humble/share/realsense2_description/meshes/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
- link right_camera_link: geometry collision box size=0.02505 0.09 0.025; visual mesh filename=file:///opt/ros/humble/share/realsense2_description/meshes/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
Joints:
- added joint left_grasp_point_joint: type fixed, parent left_tool0, child left_grasp_point, origin xyz=0 0 0.15 rpy=0 0 0
- added joint right_grasp_point_joint: type fixed, parent right_tool0, child right_grasp_point, origin xyz=0 0 0.15 rpy=0 0 0
- joint left_base_joint: origin xyz=0.0 0.5 1.0 rpy=0.0 0.0 0.0 -> xyz=0.0 0.5 1.02 rpy=0.0 0.0 0.0
- joint right_base_joint: origin xyz=0.0 -0.5 1.0 rpy=0.0 0.0 0.0 -> xyz=0.0 -0.5 1.02 rpy=0.0 0.0 0.0

File: src/robot_setup/ur_ft_description/urdf/test.urdf (robot description, URDF)
Before this commit: robot ur_ft, 17 links, 16 joints
Links:
- added link tip_link_end
Joints:
- added joint tip_link_end_joint: type fixed, parent tip_link, child tip_link_end, origin xyz=0 0 0.06 rpy=0 0 0
- joint base_joint: origin xyz=0.0 0.0 1.0 rpy=0.0 0.0 0.0 -> xyz=0.0 0.0 1.0 rpy=0.0 0.0 -1.5707

File: src/robot_setup/ur_ft_description/urdf/ur_ft.urdf.xacro (robot description, xacro)
@@ -13,5 +13,5 @@
     <xacro:include filename="$(find ur_ft_description)/urdf/ur_ft_macro.urdf.xacro"/>
     <link name="world"/>
-    <!-- robot: ur_ft -->
+    <!-- robot ur_ft -->
     <xacro:ur_ft
         ur_name="ur"

File: src/robot_setup/ur_robotiq_rs_description/urdf/test.urdf (robot description, URDF)
Before this commit: robot ur_robotiq_rs, 39 links, 38 joints
Links:
- added link grasp_point
Joints:
- added joint grasp_point_joint: type fixed, parent tool0, child grasp_point, origin xyz=0 0 0.15 rpy=0 0 0
- joint base_joint: origin xyz=0 0.5 1.03 rpy=0 0 0 -> xyz=0.0 0.0 1.0 rpy=0.0 0.0 1.5707
